File: Hardware/temaTSC.sch (EAGLE design)
At the start: 105 parts, among them IC1 BQ25180YBGR_BQ25180YBGR, IC2 DRV2605YZFR_DRV2605YZFR, IC3 BMA423_BMA423, IC9 RT6160AWSC_RT6160AWSC, J1 503480-2400_503480-2400, J2 TC2030-IDC_TC2030-IDC, J4 KH-TYPE-C-16P_KH-TYPE-C-16P, Q2 20V/4.2A/52mΩ/1.4W, Q3 ESP32_C6_LIBRARY_6_SI1308EDL-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, U1 NRF52840_QF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

Commit message: schematic dupa review
Parts:
- removed C27: 0.1uF, InkTime_v5:NORDIC_NRF_3_CAPACITOR_0201_L
- added C26: 0.1uF, InkTime_v5:GRM011R60J152KE01L_1_GRM011R60J152KE01L
- C29, C30, C31, C34: device InkTime_v5:NORDIC_NRF_3_CAPACITOR_0201_L -> InkTime_v5:GRM011R60J152KE01L_1_GRM011R60J152KE01L
- C32: device InkTime_v5:NORDIC_NRF_3_CAPACITOR_0402_L -> InkTime_v5:GRM011R60J152KE01L_1_GRM011R60J152KE01L
- renumbered Q2 to Q1
Connections:
- removed net N$29: EPD_C5.2, J1.15, J1.16
- net 3V3/1.7D: now also C34.2; no longer C34.1
- net EPD_3V3: now also EPD_C5.2, J1.15, J1.16
- net GND: now also C26.1, C29.1, C30.1, C31.1, C32.1, C34.1; no longer C27.2, C29.2, C30.2, C31.2, C32.2, C34.2
- net N$32: now also C32.2; no longer C32.1
- net P0.13/1.5D: now also C30.2; no longer C30.1
- net P0.14/1.5D: now also C31.2; no longer C31.1
- net P1.02/1.6C: now also C29.2; no longer C29.1
- net VBAT/1.2A: now also C26.2; no longer C27.1
