File: Hardware/temaTSCpcb.brd (EAGLE design)
At the start: 46 x 35 mm, 105 parts, among them IC1 BQ25180YBGR_BQ25180YBGR, IC2 DRV2605YZFR_DRV2605YZFR, IC3 BMA423_BMA423, IC9 RT6160AWSC_RT6160AWSC, J1 503480-2400_503480-2400, J2 TC2030-IDC_TC2030-IDC, J4 KH-TYPE-C-16P_KH-TYPE-C-16P, Q2 20V/4.2A/52mΩ/1.4W, Q3 ESP32_C6_LIBRARY_6_SI1308EDL-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, U1 NRF52840_QF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

Commit message: pcb dupa review
Parts:
- removed C27: 0.1uF, InkTime_v5:NORDIC_NRF_3_RESC0201_L
- added C26: 0.1uF, InkTime_v5:GRM011R60J152KE01L_1_0201
- C29, C30, C31, C34: device InkTime_v5:NORDIC_NRF_3_RESC0201_L -> InkTime_v5:GRM011R60J152KE01L_1_0201
- C32: device InkTime_v5:NORDIC_NRF_3_RESC0402_L -> InkTime_v5:GRM011R60J152KE01L_1_0201
- moved C34 21.5 mm to (27.4, 69.3), turned to 90 degrees
- moved C29 4.89 mm to (35.0, 65.4), turned to 90 degrees
- moved C31 2.72 mm to (26.9, 67.3)
- moved C30 2.67 mm to (15.5, 68.8)
- moved C32 0.37 mm to (48.1, 73.1)
- moved SW_UP 0.10 mm to (18.1, 65.7)
- renumbered Q2 to Q1
Connections:
- removed net N$29: EPD_C5.2, J1.15, J1.16
- net 3V3/1.7D: now also C34.2; no longer C34.1
- net EPD_3V3: now also EPD_C5.2, J1.15, J1.16
- net GND: now also C26.1, C29.1, C30.1, C31.1, C32.1, C34.1; no longer C27.2, C29.2, C30.2, C31.2, C32.2, C34.2
- net N$32: now also C32.2; no longer C32.1
- net P0.13/1.5D: now also C30.2; no longer C30.1
- net P0.14/1.5D: now also C31.2; no longer C31.1
- net P1.02/1.6C: now also C29.2; no longer C29.1
- net VBAT/1.2A: now also C26.2; no longer C27.1
Routing:
- net GND: track 60.1 -> 55.0 mm
- net EPD_3V3: track 36.4 -> 41.0 mm
- net N$29: track 2.41 -> 0.00 mm
- net P0.13/1.5D: track 12.9 -> 14.0 mm
- net P0.14/1.5D: track 3.73 -> 4.63 mm
- net 3V3/1.7D: track 34.5 -> 35.3 mm
- net VBAT/1.2A: track 9.29 -> 10.0 mm

Commit message: Add files via upload
Parts:
- moved ANT1 3.02 mm to (49.8, 78.3)
Routing:
- net SWDIO: track 28.6 -> 24.5 mm
- net RF: track 8.04 -> 11.1 mm
- net SWDCLK: track 27.3 -> 29.2 mm, vias 0 -> 2
Other:
- board size 46 x 35 mm -> 46.1 x 35 mm
